Commit message: Fix torso mass to 40 kg in URDF/MJCF, remove runtime overrides
- Corrected URDF and MJCF torso mass from 0.627 kg to 40 kg with
  proportionally scaled inertia (total robot mass now 71.1 kg)
- Removed runtime mass override from simulation_loop.py, sim_torso6d.py,
  and sim_lutze.py — mass is now set at the model level only
- Added assertion verifying torso mass matches 40 kg at init
- Re-tuned settling (n_settle_steps=500) and EXT gain (ext_Kd_ee=22)
  to achieve 3/3 docks after mass correction
- Result: 3/3 docks (3.3, 4.8, 4.8 mm), peak L_com=15.65 Nms

https://claude.ai/code/session_01Q7PBtNJgiGzZjqXUUeJhWJ

File: models/VISPA_crawling_fixed.urdf (robot description, URDF)
Before this commit: robot VISPA, 16 links, 15 joints
Links:
- link Link_0: mass 0.627 -> 40.0

Commit message: 7-DOF arms: add SEW elbow-swivel joint (spec §4.9.6)
Add a 7th joint per arm between Joint_2 and Joint_3, axis along the
shoulder→elbow direction (Link_2's x-axis). This matches the standard
7-DOF VISPA layout from the MIRROR project (Mishra et al., 2022) and
gives the swing EE task a 2-DOF null space during single-support —
the minimum needed to control both position and orientation against
an anchor while keeping one arm as stance.

Model changes
-------------
* models/VISPA_crawling_fixed.urdf
  - New link Link_2_swivel_{a,b} (near-massless, 1 mg, 1e-6 inertia).
  - New revolute joint Joint_swivel_{a,b}: parent=Link_2_{a,b},
    child=Link_2_swivel_{a,b}, origin=(0.5, 0, 0), axis=(1, 0, 0),
    effort=50, range=±π. Joint_3 parent changes to the new swivel
    link with origin=(0,0,0) rpy=(0,0,-π/2).
  - nq 19 → 21, nv 18 → 20, n_joints 12 → 14.

* models/VISPA_crawling_rwa3.xml (and the three 8pct variants)
  - New intermediate body Link_2_swivel_{a,b} inside Link_2_{a,b},
    pos=(0.5, 0, 0), holding the swivel joint and a tiny inertia.
  - New actuators act_SWa / act_SWb ordered to match pinocchio
    joint order: J1a J2a SW_a J3a J4a J5a J6a  J1b J2b SW_b J3b J4b J5b J6b.
  - Keyframe home qpos bumped from 12 to 14 arm zeros.
  - Doc block updated: nq=31, nv=29, nu=17, ctrl[14:17]=RWA.

Code changes
------------
* crawlbot/core/robot_interface.py, state_conversions.py
  — already DOF-generic via _detect_arm_slices() and length-based
  infer_n_joints(); no code change needed. At load, nq=21 nv=20
  n_joints=14 arm_a_v_slice=[6,13) arm_b_v_slice=[13,20) — verified.

* crawlbot/simulation/sim_loop.py
  - _diag_lock_arm_joints: replace the hardcoded qvel[15:27] slice
    with a dynamic `arm_v_start = 6 + (3 if has_rwa else 0) + 6`
    and length = self.robot.n_joints.

* crawlbot/diagnostics/plots.py
  - _to_np2d: when numpy stacks a list of per-step 1D arrays into a
    2D array directly, trust the inner dimension instead of the
    fallback cols=3/12 hint. Fixes fig7 crash on 14-wide tau arrays.

* tests/test_invariants.py
  - Replace hardcoded np.zeros(18) / np.random.randn(18) with
    robot_interface.model.nv.
  - Shape assertions on contact Jacobians use model.nv instead of 18.
  - (12, nv) contact-wrench shape stays 12 because 12 = 2·6, not
    joint count.

Test suite: 191/191 pass.

1% single-step result (dock gate: d<5mm AND ori<5°)
---------------------------------------------------
- 0 dock events (same as the 6-DOF-with-gate run).
- Step 0 SS+EXT window: 162 samples
- Min d = 41.60 mm at t=8.40s; ori at that moment = 4.22° — UNDER
  the 5° budget, which was impossible with 6-DOF arms.
- Min ori overall = 0.07° (pre-motion, d=800 mm).
- **20/162 samples with ori < 5°** — the 7-DOF arm is actively
  meeting the orientation budget (was 0/162 with 6-DOF).
- Among ori<5° samples, the best d was 41.60 mm.
- 0/162 samples with both d<5mm AND ori<5° simultaneously.
- Close-approach band d<100 mm: 24 samples, ori range [3.01°,69.70°].
- Platform rotation 6.22° (slightly over 5°), NMPC solve rate 100%,
  NMPC infeasibility 0%, hw_peak 0.82.

Interpretation
--------------
The kinematic deficit from spec §2 is FIXED: the arm can now bring
its orientation under 5° at close range (20 samples demonstrate it).
The remaining issue is a control-trajectory stall: between t=8.1 and
t=8.4 s the gripper reaches d≈41 mm with ori≈4°, but the torso
quintic is still accelerating (45 % progress of its 1.7–16.5 s run)
and drags the swing arm away: d goes 41 → 97 mm over the next 0.9 s
while ori grows 4° → 18°. The close-approach latch fires at d<20 mm,
which is never reached, so the torso never freezes.

This is a CONTROL-TUNING problem, not a kinematic one — likely needs
either (a) a larger close-approach threshold (d<50 mm) to freeze the
torso once the arm is "close enough", (b) higher EE-position gains,
or (c) a re-parameterized torso trajectory that is already resting
by the time EXT starts. That is the next conversation.

https://claude.ai/code/session_019icSadYAqoNSWQ93buum8q

File: models/VISPA_crawling_fixed.urdf (robot description, URDF)
Before this commit: robot VISPA, 16 links, 15 joints
Links:
- added link Link_2_swivel_a, mass 0.001
- added link Link_2_swivel_b, mass 0.001
Joints:
- added joint Joint_swivel_a: type revolute, parent Link_2_a, child Link_2_swivel_a, origin xyz=0.5 0 0 rpy=0 0 0, axis 1 0 0, limit lower=-3.14159265359 upper=3.14159265359 effort=50 velocity=0.09395689
- added joint Joint_swivel_b: type revolute, parent Link_2_b, child Link_2_swivel_b, origin xyz=0.5 0 0 rpy=0 0 0, axis 1 0 0, limit lower=-3.14159265359 upper=3.14159265359 effort=50 velocity=0.09395689
- joint Joint_3_a: origin xyz=0.5 0 0 rpy=0 0 -1.57079632679 -> xyz=0 0 0 rpy=0 0 -1.57079632679; parent Link_2_a -> Link_2_swivel_a
- joint Joint_3_b: origin xyz=0.5 0 0 rpy=0 0 -1.57079632679 -> xyz=0 0 0 rpy=0 0 -1.57079632679; parent Link_2_b -> Link_2_swivel_b
